File: Fatbot/sch.sch (EAGLE design)
At the start: 85 parts, among them IC1 LM317MBSTT3, Q1 FZT788B, Q2 NPN, Q3 NPN, Q4 NPN, Q5 NPN, U2 DRV8871, U3 BQ2057WSN, U4 MAX1704X, U5 LSM9DS1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

Commit message: add image
Other:
- note added: "TODO: Test points"
Changed lines of the file:
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@@
 <text x="261.62" y="134.62" size="1.778" layer="97">9DOF SENSOR</text>
 <text x="5.08" y="137.16" size="1.778" layer="97">2C_BATTERY_CHARGER</text>
+<text x="299.72" y="-17.78" size="1.778" layer="91">TODO: Test points</text>
 </plain>
 <instances>

Commit message: shit
Parts:
- removed R11: 4.7k, SparkFun:RESISTOR0402-RES
- added R2: 4.7k, SparkFun:RESISTOR0402-RES
- BATTERY, CHARGER, EMER_SWITCH, MY_RIO_POWER, MY_RIO_SWITCH: device SparkFun-Connectors:M02-JST-2-PTH-NO_SILK -> SparkFun-Connectors:CONN_02
- renumbered VL53L0X1 to ULTRA_1, VL53L0X2 to ULTRA_2
Connections:
- net SDA: now also R2.1; no longer R11.1
- net V_BATT: now also R2.2; no longer R11.2
