File: Power Dis v2.2/untitled.sch (EAGLE design)
At the start: 77 parts, among them J1 PCIE-098-02-X-D-TH, Q1 MMBT2222, U1 MCP9808MSOP, U2 ADS1115IDGST

Commit message: shit
Parts:
- removed 24V, AUX4: (no value), SparkFun-Connectors:CONN_02
- removed C5, C6: 0.1uF, SparkFun-Capacitors:0.1UF-0603-25V-(+80/-20%)
- removed J1: PCIE-098-02-X-D-TH, PCIE-098-02-X-D-TH:PCIE-098-02-X-D-TH
- removed R11: 10k, SparkFun-Resistors:10KOHM-0603-1/10W-1%
- removed R12: 2.0k, SparkFun-Resistors:2.0KOHM-0603-1/10W-5%
- removed SUPER_CAP, TO_CAP_24V: XT60, NewKevinMade:XT60
- removed VR2: 10k, SparkFun-Resistors:TRIMPOT-SMD-3MM-OPEN-1/10W-25%
- added 24V_AUX, 24V_AUX2: XT30, NewKevinMade:XT30
- added TO_CAP_26V, TO_CAP_BOARD, TO_CAP_REAL, TO_MOTOR: XT60PW-M, XT60PW-M:XT60PW-M
- AUX_BAT: value XT60 -> XT60PW-M; device NewKevinMade:XT60 -> XT60PW-M:XT60PW-M
- renumbered U$7 to RELAY
Connections:
- net CANH renamed CAN_H
- net CANL renamed CAN_L
- net CHARGE_OR_NOT renamed AUX_DIGI
- removed net CAP_ANALOG_OUT: C5.2, C6.1, R11.1, R12.2, U2.AIN2
- removed net N$10: J1G$1.7, J1G$1.8
- removed net N$11: J1G$1.10, J1G$1.11, J1G$1.9
- removed net N$16: J1G$1.12, J1G$1.13, J1G$1.14, J1G$1.15, J1G$1.16, J1G$1.17, J1G$1.18, J1G$1.19, J1G$1.20, J1G$1.21, J1G$1.22
- removed net N$18: J1G$1.35, J1G$1.36, J1G$1.37, J1G$1.38, J1G$1.39, J1G$1.40, J1G$1.41, J1G$1.42, J1G$1.43, J1G$1.44, J1G$1.45, J1G$1.46, J1G$1.47, J1G$1.48, J1G$1.49
- removed net N$19: J1G$1.23, J1G$1.24, J1G$1.25, J1G$1.26, J1G$1.27, J1G$1.28, J1G$1.29, J1G$1.30, J1G$1.31, J1G$1.32, J1G$1.33, J1G$1.34
- removed net N$2: J1G$1.1, J1G$1.2
- removed net N$3: J1G$1.3, J1G$1.4
- removed net N$6: C5.1, R11.2, VR2.WIPER
- removed net N$9: J1G$1.5, J1G$1.6
- new net CAP_MOTOR_24V: AUX_CAP_POW.VCC, MOTOR1.VCC, MOTOR2.VCC, MOTOR3.VCC, MOTOR4.VCC, RELAYG$1.S, TO_MOTOR.1
- net 5V_AUX: no longer AUX4.1
- net BAT_24V: now also 24V_AUX.VCC, 24V_AUX2.VCC, AUX_BAT.2, TO_CAP_26V.1; no longer 24V.2, AUX_BAT.VCC, TO_CAP_24V.VCC
- net BAT_GND: now also 24V_AUX.GND, 24V_AUX2.GND, AUX_BAT.1, TO_CAP_26V.2, TO_CAP_BOARD.2, TO_CAP_REAL.1, TO_MOTOR.2; no longer 24V.1, AUX4.2, AUX_BAT.GND, C6.2, R12.1, SUPER_CAP.GND, TO_CAP_24V.GND, VR2.CW
- net CAP_24V: now also TO_CAP_BOARD.1, TO_CAP_REAL.2; no longer AUX_CAP_POW.VCC, MOTOR1.VCC, MOTOR2.VCC, MOTOR3.VCC, MOTOR4.VCC, RELAYG$1.S, SUPER_CAP.VCC, VR2.CCW
