File: Robomaster V3.0 Controller Board/untitled.brd (EAGLE design)
At the start: 51.3 x 81.9 mm, 66 parts, among them IC1 CP2104, IC2 MCP23008/SO, IC3 PCF8523T, Q1 mmbt2222, Q2 mmbt2222, Q3 DMG3415U, SW2 KMR2, U1 TCA9548APWR, U2 AP2112-3.3, X1 microsd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

Commit message: shit
Parts:
- renumbered I2C_AUX1 to I2C_HUD, I2C_SCREEN to I2C_OLED, TO_HUD to TO_SUPER_CAP
Connections:
- removed net A0_DAC2: X2.11
- removed net IO27_A10: X2.12
- new net RX_CUS: TO_SUPER_CAP.1, X2.12
- new net TX_CUS: TO_SUPER_CAP.2, X2.11
- net 2RX: no longer TO_SUPER_CAP.1
- net 2TX: no longer TO_SUPER_CAP.2
Routing:
- net TX_CUS: track 0.00 -> 34.1 mm, vias 0 -> 3
- net RX_CUS: track 0.00 -> 30.9 mm, vias 0 -> 2
- net 2TX: track 20.8 -> 18.4 mm
- net 2RX: track 26.0 -> 24.7 mm
- net N$6: track 10.9 -> 10.3 mm
Other:
- board text added: "ROBOMASTER CONTROLLER V3.1 BY CHENGMING ZHANG 4.1.2019.2AM / 4 LAYER 7.16,2019.9PM / 4 LAYER"
- board text removed: "ROBOMASTER CONTROLLER V3.0 BY CHENGMING ZHANG 4.1.2019.2AM / 4 LAYER"
