File: Robomaster V3.0 Controller Board/untitled.sch (EAGLE design)
At the start: 66 parts, among them IC1 CP2104, IC2 MCP23008/SO, IC3 PCF8523T, Q1 mmbt2222, Q2 mmbt2222, Q3 DMG3415U, SW2 KMR2, U1 TCA9548APWR, U2 AP2112-3.3, X1 microsd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

Commit message: shit
Parts:
- renumbered I2C_AUX1 to I2C_HUD, I2C_SCREEN to I2C_OLED, TO_HUD to TO_SUPER_CAP
Connections:
- removed net A0_DAC2: X2.IO26/DAC2/A2_9
- removed net IO27_A10: X2.IO27/A2_7
- new net RX_CUS: TO_SUPER_CAP.JST1, X2.IO27/A2_7
- new net TX_CUS: TO_SUPER_CAP.JST2, X2.IO26/DAC2/A2_9
- net 2RX: no longer TO_SUPER_CAP.JST1
- net 2TX: no longer TO_SUPER_CAP.JST2
Other:
- note added: "CHARGE OR NOT NOT DEFINED"
- note removed: "TODO: CHANGE OLED TO RM OLED (SPI)"
Changed lines of the file:
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@@
 <part name="GND4" library="SparkFun-Aesthetics" deviceset="GND" device=""/>
 <part name="TO_STM32" library="NewKevinMade" deviceset="S3B-PH-SM4_TB" device=""/>
-<part name="TO_HUD" library="NewKevinMade" deviceset="S3B-PH-SM4_TB" device=""/>
+<part name="TO_SUPER_CAP" library="NewKevinMade" deviceset="S3B-PH-SM4_TB" device=""/>
 <part name="X1" library="microbuilder" deviceset="MICROSD" device="" value="microsd"/>
 <part name="GND10" library="supply1" deviceset="GND" device=""/>
 <part name="R17" library="microbuilder" deviceset="RESISTOR" device="_0603_NOOUT" value="100K"/>
 <part name="SJ1" library="microbuilder" deviceset="SOLDERJUMPER_CLOSED" device=""/>
-<part name="I2C_SCREEN" library="NewKevinMade" deviceset="S4B-PH-SM4_TB" device=""/>
+<part name="I2C_OLED" library="NewKevinMade" deviceset="S4B-PH-SM4_TB" device=""/>
 <part name="GND11" library="SparkFun-Aesthetics" deviceset="GND" device=""/>
 <part name="TO_ELE_DIS" library="NewKevinMade" deviceset="S6B-PH-SM4_TB" device=""/>
-<part name="I2C_AUX1" library="NewKevinMade" deviceset="S4B-PH-SM4_TB" device=""/>
+<part name="I2C_HUD" library="NewKevinMade" deviceset="S4B-PH-SM4_TB" device=""/>
 <part name="GND12" library="SparkFun-Aesthetics" deviceset="GND" device=""/>
 <part name="I2C_AUX2" library="NewKevinMade" deviceset="S4B-PH-SM4_TB" device=""/>
@@
 VBAT SENSE: IO35
 LED: IO13</text>
-<text x="154.94" y="22.86" size="1.778" layer="95">TODO: CHANGE OLED TO RM OLED (SPI)</text>
+<text x="154.94" y="22.86" size="1.778" layer="95">CHARGE OR NOT NOT DEFINED</text>
 </plain>
 <instances>
@@
 <attribute name="NAME" x="342.9" y="102.108" size="1.778" layer="95"/>
 </instance>
-<instance part="TO_HUD" gate="G$1" x="340.36" y="53.34" smashed="yes">
+<instance part="TO_SUPER_CAP" gate="G$1" x="340.36" y="53.34" smashed="yes">
 <attribute name="NAME" x="342.9" y="74.168" size="1.778" layer="95"/>
 </instance>
@@
 <attribute name="VALUE" x="227.33" y="134.62" size="1.778" layer="96" rot="R90"/>
 </instance>
-<instance part="I2C_SCREEN" gate="G$1" x="375.92" y="78.74" smashed="yes">
+<instance part="I2C_OLED" gate="G$1" x="375.92" y="78.74" smashed="yes">
 <attribute name="NAME" x="378.46" y="102.108" size="1.778" layer="95"/>
 </instance>
@@
 <attribute name="NAME" x="342.9" y="43.688" size="1.778" layer="95"/>
 </instance>
-<instance part="I2C_AUX1" gate="G$1" x="375.92" y="50.8" smashed="yes">
+<instance part="I2C_HUD" gate="G$1" x="375.92" y="50.8" smashed="yes">
 <attribute name="NAME" x="378.46" y="74.168" size="1.778" layer="95"/>
 </instance>
@@
 <wire x1="337.82" y1="58.42" x2="337.82" y2="53.34" width="0.1524" layer="91"/>
 <pinref part="GND3" gate="1" pin="GND"/>
-<pinref part="TO_HUD" gate="G$1" pin="JST3"/>
-<pinref part="TO_HUD" gate="G$1" pin="GND*"/>
+<pinref part="TO_SUPER_CAP" gate="G$1" pin="JST3"/>
+<pinref part="TO_SUPER_CAP" gate="G$1" pin="GND*"/>
 </segment>
 <segment>
@@
 </segment>
 <segment>
-<pinref part="I2C_SCREEN" gate="G$1" pin="JST4"/>
+<pinref part="I2C_OLED" gate="G$1" pin="JST4"/>
 <wire x1="375.92" y1="91.44" x2="373.38" y2="91.44" width="0.1524" layer="91"/>
 <wire x1="373.38" y1="91.44" x2="373.38" y2="83.82" width="0.1524" layer="91"/>
-<pinref part="I2C_SCREEN" gate="G$1" pin="GND*"/>
+<pinref part="I2C_OLED" gate="G$1" pin="GND*"/>
 <wire x1="373.38" y1="83.82" x2="375.92" y2="83.82" width="0.1524" layer="91"/>
 <wire x1="373.38" y1="83.82" x2="373.38" y2="81.28" width="0.1524" layer="91"/>
@@
 </segment>
 <segment>
-<pinref part="I2C_AUX1" gate="G$1" pin="JST4"/>
+<pinref part="I2C_HUD" gate="G$1" pin="JST4"/>
 <wire x1="375.92" y1="63.5" x2="373.38" y2="63.5" width="0.1524" layer="91"/>
 <wire x1="373.38" y1="63.5" x2="373.38" y2="55.88" width="0.1524" layer="91"/>
-<pinref part="I2C_AUX1" gate="G$1" pin="GND*"/>
+<pinref part="I2C_HUD" gate="G$1" pin="GND*"/>
 <wire x1="373.38" y1="55.88" x2="375.92" y2="55.88" width="0.1524" layer="91"/>
 <wire x1="373.38" y1="55.88" x2="373.38" y2="53.34" width="0.1524" layer="91"/>
@@
 </segment>
 </net>
-<net name="A0_DAC2" class="1">
+<net name="TX_CUS" class="1">
 <segment>
 <wire x1="78.74" y1="76.2" x2="91.44" y2="76.2" width="0.1524" layer="91"/>
@@
 <pinref part="X2" gate="G$1" pin="IO26/DAC2/A2_9"/>
 </segment>
+<segment>
+<wire x1="340.36" y1="68.58" x2="337.82" y2="68.58" width="0.1524" layer="91"/>
+<pinref part="TO_SUPER_CAP" gate="G$1" pin="JST2"/>
+<label x="335.28" y="68.58" size="1.778" layer="95"/>
+</segment>
 </net>
 <net name="2RX" class="1">
@@
 <label x="335.28" y="99.06" size="1.778" layer="95"/>
 </segment>
-<segment>
-<wire x1="340.36" y1="71.12" x2="337.82" y2="71.12" width="0.1524" layer="91"/>
-<pinref part="TO_HUD" gate="G$1" pin="JST1"/>
-<label x="335.28" y="71.12" size="1.778" layer="95"/>
-</segment>
 </net>
 <net name="2TX" class="1">
@@
 <pinref part="TO_STM32" gate="G$1" pin="JST2"/>
 <label x="335.28" y="96.52" size="1.778" layer="95"/>
-</segment>
-<segment>
-<wire x1="340.36" y1="68.58" x2="337.82" y2="68.58" width="0.1524" layer="91"/>
-<pinref part="TO_HUD" gate="G$1" pin="JST2"/>
-<label x="335.28" y="68.58" size="1.778" layer="95"/>
 </segment>
 </net>
@@
 </segment>
 <segment>
-<pinref part="I2C_SCREEN" gate="G$1" pin="JST2"/>
+<pinref part="I2C_OLED" gate="G$1" pin="JST2"/>
 <wire x1="375.92" y1="96.52" x2="373.38" y2="96.52" width="0.1524" layer="91"/>
 <label x="373.38" y="96.52" size="1.778" layer="95" rot="R180"/>
@@
 </segment>
 <segment>
-<pinref part="I2C_AUX1" gate="G$1" pin="JST2"/>
+<pinref part="I2C_HUD" gate="G$1" pin="JST2"/>
 <wire x1="375.92" y1="68.58" x2="373.38" y2="68.58" width="0.1524" layer="91"/>
 <label x="373.38" y="68.58" size="1.778" layer="95" rot="R180"/>
@@
 </segment>
 <segment>
-<pinref part="I2C_SCREEN" gate="G$1" pin="JST3"/>
+<pinref part="I2C_OLED" gate="G$1" pin="JST3"/>
 <wire x1="375.92" y1="93.98" x2="373.38" y2="93.98" width="0.1524" layer="91"/>
 <label x="373.38" y="93.98" size="1.778" layer="95" rot="R180"/>
@@
 </segment>
 <segment>
-<pinref part="I2C_AUX1" gate="G$1" pin="JST3"/>
+<pinref part="I2C_HUD" gate="G$1" pin="JST3"/>
 <wire x1="375.92" y1="66.04" x2="373.38" y2="66.04" width="0.1524" layer="91"/>
 <label x="373.38" y="66.04" size="1.778" layer="95" rot="R180"/>
@@
 </segment>
 </net>
-<net name="IO27_A10" class="1">
+<net name="RX_CUS" class="1">
 <segment>
 <wire x1="78.74" y1="73.66" x2="91.44" y2="73.66" width="0.1524" layer="91"/>
 <label x="81.28" y="73.66" size="1.778" layer="95"/>
 <pinref part="X2" gate="G$1" pin="IO27/A2_7"/>
+</segment>
+<segment>
+<wire x1="340.36" y1="71.12" x2="337.82" y2="71.12" width="0.1524" layer="91"/>
+<pinref part="TO_SUPER_CAP" gate="G$1" pin="JST1"/>
+<label x="335.28" y="71.12" size="1.778" layer="95"/>
 </segment>
 </net>
@@
 </segment>
 <segment>
-<pinref part="I2C_SCREEN" gate="G$1" pin="JST1"/>
+<pinref part="I2C_OLED" gate="G$1" pin="JST1"/>
 <wire x1="375.92" y1="99.06" x2="373.38" y2="99.06" width="0.1524" layer="91"/>
 <label x="373.38" y="99.06" size="1.778" layer="95" rot="R180"/>
 </segment>
 <segment>
-<pinref part="I2C_AUX1" gate="G$1" pin="JST1"/>
+<pinref part="I2C_HUD" gate="G$1" pin="JST1"/>
 <wire x1="375.92" y1="71.12" x2="373.38" y2="71.12" width="0.1524" layer="91"/>
 <label x="373.38" y="71.12" size="1.778" layer="95" rot="R180"/>
